Commit message: 2026 06.09 10：32

File: src/wtb_car_driver/urdf/wtb_car.xacro (robot description, xacro)
@@ -104,9 +104,7 @@
         <joint name="lidar_joint" type="fixed">
             <parent link="base_link" />
-            <!-- <child link="laser_link" />   -->
             <child link="laser" />
             <origin xyz="${lidar_x} ${lidar_y} ${lidar_z}" rpy="0 0 0" />
         </joint>
-        <!-- <link name="laser_link"> -->
         <link name="laser">
             <visual>

File: src/wvcsc_sensor_kit_launch/wvcsc_sensor_kit_description/urdf/sensor_kit.xacro (robot description, xacro)
@@ -48,21 +48,4 @@
       </visual>
     </link>
-    <joint name="gnss_link_joint" type="fixed">
-      <origin
-        xyz="${calibration['sensor_kit_base_link']['gnss_link']['x']} ${calibration['sensor_kit_base_link']['gnss_link']['y']} ${calibration['sensor_kit_base_link']['gnss_link']['z']}"
-        rpy="${calibration['sensor_kit_base_link']['gnss_link']['roll']} ${calibration['sensor_kit_base_link']['gnss_link']['pitch']} ${calibration['sensor_kit_base_link']['gnss_link']['yaw']}"
-      />
-      <parent link="${sensor_kit_base_link}"/>
-      <child link="gnss_link"/>
-    </joint>
-    <link name="gnss_link">
-      <visual>
-        <origin xyz="0 0 0" rpy="0 0 0"/>
-        <geometry>
-          <box size="0.08 0.08 0.02"/>
-        </geometry>
-        <material name="gray"/>
-      </visual>
-    </link>
   </xacro:macro>
 </robot>

File: src/wvcsc_vehicle_launch/wvcsc_vehicle_description/urdf/wvcsc_vehicle_base.xacro (robot description, xacro)
@@ -19,8 +19,8 @@
       </visual>
     </link>
-    <joint name="base_link_joint" type="fixed">
-      <parent link="base_footprint"/>
-      <child link="base_link"/>
-      <origin xyz="0 0 ${base_link_to_footprint_z}" rpy="0 0 0"/>
+    <joint name="base_footprint_joint" type="fixed">
+      <parent link="base_link"/>
+      <child link="base_footprint"/>
+      <origin xyz="0 0 ${-base_link_to_footprint_z}" rpy="0 0 0"/>
     </joint>
     <link name="base_link">
