Commit message: 2026 07.14 18:13

File: src/wtb_car_driver/urdf/wtb_car.xacro (robot description, xacro)
@@ -1,143 +1,101 @@
-<?xml version="1.0" ?>
+<?xml version="1.0"?>
 <robot name="wtb_robot" xmlns:xacro="http://www.ros.org/wiki/xacro">
-    <xacro:property name="base_length" value="1.30" />
-    <xacro:property name="base_width"  value="0.80" />
-    <xacro:property name="base_height" value="1.00" />
-    <xacro:property name="base_z"      value="0.16" />
-    <xacro:property name="wheel_radius" value="0.20" />
-    <xacro:property name="wheel_length" value="0.12" />
-    <xacro:property name="wheel_z"      value="0" />
-    <xacro:property name="wheel_x"      value="0.35" />
-    <xacro:property name="lidar_radius"   value="0.08" />
-    <xacro:property name="lidar_height"   value="0.15" />
-    <xacro:property name="lidar_x"        value="0.36" />
-    <xacro:property name="lidar_y"        value="0" />
-    <xacro:property name="lidar_z_offset" value="0.0" />
-    <xacro:property name="lidar_z" value="${base_height/2 +  lidar_z_offset}" />
-    <xacro:property name="base_footprint_z" value="0.0" />
-    <xacro:property name="base_link_to_footprint_z" value="${base_z + base_height/2}" />
-    <xacro:macro name="material_white">
-        <material name="white">
-            <color rgba="1 1 1 1" />
-        </material>
-    </xacro:macro>
-    <xacro:macro name="material_black">
-        <material name="black">
-            <color rgba="0 0 0 1" />
-        </material>
-    </xacro:macro>
-    <xacro:macro name="material_gray">
-        <material name="gray">
-            <color rgba="0.5 0.5 0.5 1" />
-        </material>
-    </xacro:macro>
-    <xacro:macro name="base_footprint">
-        <link name="base_footprint">
-            <visual>
-                <origin xyz="0 0 0" rpy="0 0 0" />
-                <geometry>
-                    <box size="0.1 0.1 0.00" />
-                </geometry>
-                <material name="red">
-                    <color rgba="1 0 0 0.8" />
-                </material>
-            </visual>
-        </link>
-         <joint name="base_link_joint" type="fixed">
-            <parent link="base_footprint" />
-            <child link="base_link" />
-            <origin xyz="0 0 ${base_link_to_footprint_z}" rpy="0 0 0" />
-        </joint>
-    </xacro:macro>
-    <xacro:macro name="base_link">
-        <link name="base_link">
-            <visual>
-                <origin xyz="0 0 0" rpy="0 0 0" />
-                <geometry>
-                    <box size="${base_length} ${base_width} ${base_height}" />
-                </geometry>
-                <xacro:material_white />
-            </visual>
-        </link>
-    </xacro:macro>
-    <xacro:macro name="wheel" params="wheel_name x y">
-        <joint name="${wheel_name}_joint" type="continuous">
-            <origin xyz="${x} ${y} ${-base_height/2 + wheel_z}" rpy="1.57 0 0" />
-            <parent link="base_link" />
-            <child link="${wheel_name}_link" />
-            <axis xyz="0 1 0" />
-        </joint>
-        <link name="${wheel_name}_link">
-            <visual>
-                <origin xyz="0 0 0" rpy="0 0 0" />
-                <geometry>
-                    <cylinder radius="${wheel_radius}" length="${wheel_length}" />
-                </geometry>
-                <xacro:material_black />
-            </visual>
-        </link>
-    </xacro:macro>
-    <xacro:macro name="steer_wheel" params="wheel_name x y">
-        <joint name="${wheel_name}_joint" type="revolute">
-            <origin xyz="${x} ${y} ${wheel_z}" rpy="1.57 0 0" />
-            <parent link="base_link" />
-            <child link="${wheel_name}_link" />
-            <axis xyz="0 0 1" />
-            <limit
-                effort="100"
-                velocity="2.0"
-                lower="-0.6109"
-                upper="0.6109"
-            />
-        </joint>
-        <link name="${wheel_name}_link">
-            <visual>
-                <origin xyz="0 0 0" rpy="0 0 0" />
-                <geometry>
-                    <cylinder radius="${wheel_radius}" length="${wheel_length}" />
-                </geometry>
-                <xacro:material_black />
-            </visual>
-        </link>
-    </xacro:macro>
-    <xacro:macro name="lidar">
-        <joint name="lidar_joint" type="fixed">
-            <parent link="base_link" />
-            <child link="laser" />
-            <origin xyz="${lidar_x} ${lidar_y} ${lidar_z}" rpy="0 0 0" />
-        </joint>
-        <link name="laser">
-            <visual>
-                <origin xyz="0 0 0" rpy="0 0 0" />
-                <geometry>
-                    <cylinder radius="${lidar_radius}" length="${lidar_height}" />
-                </geometry>
-                <xacro:material_gray />
-            </visual>
-        </link>
-    </xacro:macro>
-    <xacro:macro name="imu">
-        <joint name="IMU_joint" type="fixed">
-            <parent link="base_link" />
-            <child link="gyro_link" />
-            <origin xyz="0 0 ${-base_height/2 +  0.1}" rpy="0 0 0"/>
-        </joint>
-        <link name="gyro_link">
-            <visual>
-                <origin xyz="0 0 0" rpy="0 0 0" />
-                <geometry>
-                    <box size="0.1 0.1 0.00" />
-                </geometry>
-                <xacro:material_gray />
-            </visual>
-        </link>
-    </xacro:macro>
-    <xacro:base_footprint />
-    <xacro:base_link />
-    <xacro:wheel wheel_name="left_front"    x="${wheel_x}"  y="0.43" />
-    <xacro:wheel wheel_name="right_wheel"   x="${-wheel_x}" y="-0.43" />
-    <xacro:wheel wheel_name="left_wheel"    x="${-wheel_x}"  y="0.43" />
-    <xacro:wheel wheel_name="right_front"   x="${wheel_x}"  y="-0.43" />
-    <xacro:lidar />
-    <xacro:imu />
+  <xacro:property name="base_length" value="1.30"/>
+  <xacro:property name="base_width" value="0.80"/>
+  <xacro:property name="base_height" value="1.00"/>
+  <xacro:property name="base_z" value="0.20"/>
+  <xacro:property name="wheel_radius" value="0.20"/>
+  <xacro:property name="wheel_length" value="0.12"/>
+  <xacro:property name="wheel_x" value="0.35"/>
+  <xacro:property name="wheel_y" value="0.43"/>
+  <xacro:macro name="box_inertial" params="mass x y z">
+    <inertial>
+      <mass value="${mass}"/>
+      <inertia ixx="${mass*(y*y+z*z)/12}" ixy="0" ixz="0"
+               iyy="${mass*(x*x+z*z)/12}" iyz="0"
+               izz="${mass*(x*x+y*y)/12}"/>
+    </inertial>
+  </xacro:macro>
+  <xacro:macro name="wheel_link" params="name">
+    <link name="${name}_link">
+      <visual>
+        <origin rpy="1.5708 0 0"/>
+        <geometry><cylinder radius="${wheel_radius}" length="${wheel_length}"/></geometry>
+        <material name="wtb_black"><color rgba="0.05 0.05 0.05 1"/></material>
+      </visual>
+      <collision>
+        <origin rpy="1.5708 0 0"/>
+        <geometry><cylinder radius="${wheel_radius}" length="${wheel_length}"/></geometry>
+      </collision>
+      <inertial>
+        <mass value="3.0"/>
+        <inertia ixx="0.0636" ixy="0" ixz="0" iyy="0.0636" iyz="0" izz="0.0216"/>
+      </inertial>
+    </link>
+  </xacro:macro>
+  <xacro:macro name="rear_wheel" params="name x y">
+    <xacro:wheel_link name="${name}"/>
+    <joint name="${name}_joint" type="continuous">
+      <parent link="base_link"/><child link="${name}_link"/>
+      <origin xyz="${x} ${y} ${-base_height/2}"/>
+      <axis xyz="0 1 0"/>
+      <limit effort="500" velocity="20"/>
+      <dynamics damping="0.2" friction="0.1"/>
+    </joint>
+  </xacro:macro>
+  <xacro:macro name="front_wheel" params="name x y">
+    <link name="${name}_steer_link">
+      <inertial><mass value="0.1"/><inertia ixx="0.001" ixy="0" ixz="0" iyy="0.001" iyz="0" izz="0.001"/></inertial>
+    </link>
+    <joint name="${name}_steer_joint" type="revolute">
+      <parent link="base_link"/><child link="${name}_steer_link"/>
+      <origin xyz="${x} ${y} ${-base_height/2}"/>
+      <axis xyz="0 0 1"/>
+      <limit effort="500" velocity="2" lower="-0.6109" upper="0.6109"/>
+      <dynamics damping="1"/>
+    </joint>
+    <xacro:wheel_link name="${name}"/>
+    <joint name="${name}_joint" type="continuous">
+      <parent link="${name}_steer_link"/><child link="${name}_link"/>
+      <axis xyz="0 1 0"/>
+      <limit effort="500" velocity="20"/>
+      <dynamics damping="0.2" friction="0.1"/>
+    </joint>
+  </xacro:macro>
+  <xacro:macro name="wtb_car">
+    <link name="base_footprint"/>
+    <link name="base_link">
+      <visual>
+        <geometry><box size="${base_length} ${base_width} ${base_height}"/></geometry>
+        <material name="wtb_white"><color rgba="1 1 1 1"/></material>
+      </visual>
+      <collision><geometry><box size="${base_length} ${base_width} ${base_height}"/></geometry></collision>
+      <xacro:box_inertial mass="90" x="${base_length}" y="${base_width}" z="${base_height}"/>
+    </link>
+    <joint name="base_link_joint" type="fixed">
+      <parent link="base_footprint"/><child link="base_link"/>
+      <origin xyz="0 0 ${base_z + base_height/2}"/>
+    </joint>
+    <xacro:front_wheel name="left_front" x="${wheel_x}" y="${wheel_y}"/>
+    <xacro:front_wheel name="right_front" x="${wheel_x}" y="${-wheel_y}"/>
+    <xacro:rear_wheel name="left_wheel" x="${-wheel_x}" y="${wheel_y}"/>
+    <xacro:rear_wheel name="right_wheel" x="${-wheel_x}" y="${-wheel_y}"/>
+    <link name="laser">
+      <visual><geometry><cylinder radius="0.08" length="0.15"/></geometry><material name="wtb_gray"><color rgba="0.5 0.5 0.5 1"/></material></visual>
+      <collision><geometry><cylinder radius="0.08" length="0.15"/></geometry></collision>
+      <inertial><mass value="0.5"/><inertia ixx="0.001" ixy="0" ixz="0" iyy="0.001" iyz="0" izz="0.001"/></inertial>
+    </link>
+    <joint name="lidar_joint" type="fixed">
+      <parent link="base_link"/><child link="laser"/><origin xyz="0.36 0 0.5"/>
+    </joint>
+    <link name="gyro_link">
+      <visual><geometry><box size="0.1 0.1 0.01"/></geometry><material name="wtb_gray"/></visual>
+      <collision><geometry><box size="0.1 0.1 0.01"/></geometry></collision>
+      <xacro:box_inertial mass="0.1" x="0.1" y="0.1" z="0.01"/>
+    </link>
+    <joint name="IMU_joint" type="fixed">
+      <parent link="base_link"/><child link="gyro_link"/><origin xyz="0 0 -0.4"/>
+    </joint>
+  </xacro:macro>
+  <xacro:wtb_car/>
 </robot>

Commit message: 2026 07.21 17:46

File: src/wtb_car_driver/urdf/wtb_car.xacro (robot description, xacro)
@@ -1,7 +1,7 @@
 <?xml version="1.0"?>
 <robot name="wtb_robot" xmlns:xacro="http://www.ros.org/wiki/xacro">
-  <xacro:property name="base_length" value="1.30"/>
-  <xacro:property name="base_width" value="0.80"/>
-  <xacro:property name="base_height" value="1.00"/>
+  <xacro:property name="base_length" value="1.45"/>
+  <xacro:property name="base_width" value="0.75"/>
+  <xacro:property name="base_height" value="1.35"/>
   <xacro:property name="base_z" value="0.20"/>
   <xacro:property name="wheel_radius" value="0.20"/>
@@ -87,5 +87,5 @@
     </link>
     <joint name="lidar_joint" type="fixed">
-      <parent link="base_link"/><child link="laser"/><origin xyz="0.36 0 0.5"/>
+      <parent link="base_link"/><child link="laser"/><origin xyz="0.4 0 0.725"/>
     </joint>
     <link name="gyro_link">

File: src/wvcsc_description/urdf/wvcsc_utb_alicia.urdf.xacro (robot description, xacro)
@@ -6,4 +6,27 @@
   <xacro:arg name="enable_c10_camera" default="true"/>
   <xacro:arg name="enable_c10_gazebo" default="false"/>
+    <!-- 机械臂车顶安装参数 -->
+  <!--
+    Alicia 原始 URDF 默认把机械臂底座命名为 base_link，
+    会与小车 base_link 重名，因此覆盖为 alicia_base_link。
+  -->
+  <xacro:arg name="alicia_base_link" default="alicia_base_link"/>
+  <!--
+    小车车体高度为 1.35 m，base_link 位于车体几何中心，
+    因此车顶相对 base_link 的 Z 坐标为 1.35 / 2 = 0.675 m。
+  -->
+  <xacro:arg name="vehicle_roof_z" default="0.675"/>
+  <!--
+    机械臂相对于车顶安装坐标系的位置：
+    沿 base_link 正 X 方向平移 0.10 m。
+  -->
+  <xacro:arg name="arm_mount_xyz" default="-0.20 0 0"/>
+  <!--
+    绕 Z 轴旋转 180°，使机械臂底座 X 轴方向反转，
+    同时保持机械臂 Z 轴朝上。
+  -->
+  <xacro:arg
+    name="arm_mount_rpy"
+    default="0 0 3.141592653589793"/>
   <!-- Temporary eye-in-hand extrinsics. Recalibrate after the real bracket is fixed. -->
   <xacro:arg name="c10_mount_xyz" default="-0.055 0 -0.10"/>
@@ -25,14 +48,34 @@
   <xacro:include filename="$(find alicia_m_descriptions)/urdf/Alicia_M_v1_1/Alicia_M_v1_1_follower.urdf"/>
   <xacro:include filename="$(find alicia_m_moveit_config)/config/alicia_m_v1_1_follower.ros2_control.xacro"/>
-  <link name="arm_mount_link">
-    <visual><geometry><box size="0.24 0.24 0.12"/></geometry><material name="mount_gray"><color rgba="0.3 0.3 0.3 1"/></material></visual>
-    <collision><geometry><box size="0.24 0.24 0.12"/></geometry></collision>
-    <inertial><mass value="5"/><inertia ixx="0.012" ixy="0" ixz="0" iyy="0.012" iyz="0" izz="0.012"/></inertial>
-  </link>
-  <joint name="arm_mount_joint" type="fixed">
-    <parent link="base_link"/><child link="arm_mount_link"/><origin xyz="0 0 0.56"/>
+  <!--
+    车顶安装坐标系。
+    wtb_car.xacro 中：
+      base_height = 1.35 m
+    base_link 位于车体几何中心，所以车顶位置为：
+      Z = 1.35 / 2 = 0.675 m
+  -->
+  <link name="arm_mount_link"/>
+  <joint name="arm_mount_frame_joint" type="fixed">
+    <parent link="base_link"/>
+    <child link="arm_mount_link"/>
+    <!-- arm_mount_link 原点位于小车车顶表面 -->
+    <origin
+      xyz="0 0 $(arg vehicle_roof_z)"
+      rpy="0 0 0"/>
   </joint>
+  <!--
+    机械臂与车顶安装坐标系之间的固定连接。
+    xyz="0.10 0 0"：
+      沿 base_link 正 X 方向移动 0.10 m。
+    rpy="0 0 pi"：
+      绕 Z 轴旋转 180°，机械臂底座 X 轴反向，
+      机械臂 Z 轴仍然保持朝上。
+  -->
   <joint name="alicia_mount_joint" type="fixed">
-    <parent link="arm_mount_link"/><child link="alicia_base_link"/><origin xyz="0 0 0.06"/>
+    <parent link="arm_mount_link"/>
+    <child link="$(arg alicia_base_link)"/>
+    <origin
+      xyz="$(arg arm_mount_xyz)"
+      rpy="$(arg arm_mount_rpy)"/>
   </joint>
   <link name="spray_nozzle_link"/>
