Commit message: 2026.07.22.07.17

File: src/wvcsc_calibration/xacro/calibration_arm_camera.urdf.xacro (robot description, xacro)
@@ -3,17 +3,18 @@
   <!-- Eye-in-hand calibration model: Alicia-M arm + C10 camera on a desk.
        No vehicle chassis, no controller_manager, no Ackermann.  -->
-  <xacro:arg name="alicia_base_link" default="base_link"/>
+  <xacro:arg name="alicia_base_link" default="alicia_base_link"/>
   <xacro:arg name="c10_mount_xyz" default="-0.055 0 -0.10"/>
   <xacro:arg name="c10_mount_rpy" default="0 -1.57079632679 0"/>
-  <!-- Anchor in Gazebo world so the arm does not fall through the desk -->
+  <!--
+    Keep the Gazebo model pose and the robot TF tree identical.  The desk
+    surface is at z=0.75 m and the Alicia-M mounting plane is 10 mm above it.
+    The entity is therefore spawned at the Gazebo origin; this fixed joint
+    carries the complete mounting height instead of hiding it in spawn_entity.
+  -->
   <link name="world"/>
-  <link name="base_footprint"/>
   <joint name="world_to_base" type="fixed">
     <parent link="world"/>
-    <child link="base_footprint"/>
-  </joint>
-  <joint name="base_to_base_link" type="fixed">
-    <parent link="base_footprint"/>
-    <child link="base_link"/>
+    <child link="$(arg alicia_base_link)"/>
+    <origin xyz="0 0 0.76" rpy="0 0 0"/>
   </joint>
   <!-- Alicia-M arm geometry (joint1–tool0) -->
@@ -69,8 +70,15 @@
       <pose>-0.055 0 0.05 0 -1.57079632679 0</pose>
       <camera name="c10_optical">
-        <horizontal_fov>1.8</horizontal_fov>
+        <!-- Calibration uses a deterministic 68.8 degree horizontal view:
+             the real workflow still uses its C10 camera_info calibration,
+             while the narrower benchmark view gives a 70 mm tabletop marker
+             enough pixels for the strict 3 mm URDF-extrinsic check. -->
+        <horizontal_fov>1.2</horizontal_fov>
         <image><width>1280</width><height>720</height><format>R8G8B8</format></image>
         <clip><near>0.02</near><far>300</far></clip>
-        <noise><type>gaussian</type><mean>0.0</mean><stddev>0.007</stddev></noise>
+        <!-- The calibration scene is a deterministic geometric benchmark.
+             Keep sensor noise out of the ground-truth comparison; C10 noise
+             belongs in the perception simulation, not the extrinsic oracle. -->
+        <noise><type>gaussian</type><mean>0.0</mean><stddev>0.0</stddev></noise>
       </camera>
       <plugin name="c10_camera_plugin" filename="libgazebo_ros_camera.so">

Commit message: 2026 07.22 11:29

File: src/wvcsc_calibration/xacro/calibration_arm_camera.urdf.xacro (robot description, xacro)
@@ -16,5 +16,5 @@
     <parent link="world"/>
     <child link="$(arg alicia_base_link)"/>
-    <origin xyz="0 0 0.76" rpy="0 0 0"/>
+    <origin xyz="0 0 0.75" rpy="0 0 0"/>
   </joint>
   <!-- Alicia-M arm geometry (joint1–tool0) -->

Commit message: 2026 07.22 15:18

File: src/wvcsc_calibration/xacro/calibration_arm_camera.urdf.xacro (robot description, xacro)
@@ -1,6 +1,8 @@
 <?xml version="1.0"?>
 <robot name="alicia_calibration" xmlns:xacro="http://www.ros.org/wiki/xacro">
-  <!-- Eye-in-hand calibration model: Alicia-M arm + C10 camera on a desk.
-       No vehicle chassis, no controller_manager, no Ackermann.  -->
+  <!-- LEGACY REFERENCE ONLY: Alicia-M arm + C10 camera on a desk.
+       calibration_sim.launch.py no longer starts this model because it lacks
+       the vehicle roof mount and chassis collision geometry. Keep it for
+       documented rollback/reference, not one-to-one vehicle validation. -->
   <xacro:arg name="alicia_base_link" default="alicia_base_link"/>
   <xacro:arg name="c10_mount_xyz" default="-0.055 0 -0.10"/>
@@ -24,4 +26,16 @@
   <xacro:arg name="gazebo_controllers_file" default="$(find wvcsc_description)/config/ros2_controllers.yaml"/>
   <xacro:arg name="ros2_control_plugin" default="gazebo_ros2_control/GazeboSystem"/>
+  <xacro:property name="c10_calibration" value="${xacro.load_yaml('$(find wvcsc_c10_camera)/config/c10_intrinsics.yaml')}"/>
+  <xacro:property name="c10_width" value="${c10_calibration['image_width']}"/>
+  <xacro:property name="c10_height" value="${c10_calibration['image_height']}"/>
+  <xacro:property name="c10_fx" value="${c10_calibration['camera_matrix']['data'][0]}"/>
+  <xacro:property name="c10_fy" value="${c10_calibration['camera_matrix']['data'][4]}"/>
+  <xacro:property name="c10_cx" value="${c10_calibration['camera_matrix']['data'][2]}"/>
+  <xacro:property name="c10_cy" value="${c10_calibration['camera_matrix']['data'][5]}"/>
+  <xacro:property name="c10_k1" value="${c10_calibration['distortion_coefficients']['data'][0]}"/>
+  <xacro:property name="c10_k2" value="${c10_calibration['distortion_coefficients']['data'][1]}"/>
+  <xacro:property name="c10_p1" value="${c10_calibration['distortion_coefficients']['data'][2]}"/>
+  <xacro:property name="c10_p2" value="${c10_calibration['distortion_coefficients']['data'][3]}"/>
+  <xacro:property name="c10_k3" value="${c10_calibration['distortion_coefficients']['data'][4]}"/>
   <xacro:alicia_m_v1_1_follower_ros2_control
     name="AliciaHardware"
@@ -70,11 +84,18 @@
       <pose>-0.055 0 0.05 0 -1.57079632679 0</pose>
       <camera name="c10_optical">
-        <!-- Calibration uses a deterministic 68.8 degree horizontal view:
-             the real workflow still uses its C10 camera_info calibration,
-             while the narrower benchmark view gives a 70 mm tabletop marker
-             enough pixels for the strict 3 mm URDF-extrinsic check. -->
-        <horizontal_fov>1.2</horizontal_fov>
-        <image><width>1280</width><height>720</height><format>R8G8B8</format></image>
+        <horizontal_fov>${2.0 * atan(c10_width / (2.0 * c10_fx))}</horizontal_fov>
+        <image><width>${c10_width}</width><height>${c10_height}</height><format>R8G8B8</format></image>
         <clip><near>0.02</near><far>300</far></clip>
+        <distortion>
+          <k1>${c10_k1}</k1><k2>${c10_k2}</k2><k3>${c10_k3}</k3>
+          <p1>${c10_p1}</p1><p2>${c10_p2}</p2>
+          <center>${c10_cx / c10_width} ${c10_cy / c10_height}</center>
+        </distortion>
+        <lens>
+          <intrinsics>
+            <fx>${c10_fx}</fx><fy>${c10_fy}</fy>
+            <cx>${c10_cx}</cx><cy>${c10_cy}</cy><s>0</s>
+          </intrinsics>
+        </lens>
         <!-- The calibration scene is a deterministic geometric benchmark.
              Keep sensor noise out of the ground-truth comparison; C10 noise
@@ -102,4 +123,9 @@
         <camera_name>color</camera_name>
         <frame_name>camera_color_optical_frame</frame_name>
+        <focal_length>${c10_fx}</focal_length>
+        <cx>${c10_cx}</cx><cy>${c10_cy}</cy>
+        <P_fx>${c10_fx}</P_fx><P_fy>${c10_fy}</P_fy>
+        <P_cx>${c10_cx}</P_cx><P_cy>${c10_cy}</P_cy>
+        <border_crop>false</border_crop>
       </plugin>
     </sensor>

File: src/wvcsc_description/urdf/wvcsc_utb_alicia.urdf.xacro (robot description, xacro)
@@ -6,4 +6,5 @@
   <xacro:arg name="enable_c10_camera" default="true"/>
   <xacro:arg name="enable_c10_gazebo" default="false"/>
+  <xacro:arg name="c10_noise_stddev" default="0.007"/>
   <xacro:arg name="calibration_fix_base" default="false"/>
     <!-- 机械臂车顶安装参数 -->
@@ -129,4 +130,18 @@
     </joint>
     <xacro:if value="$(arg enable_c10_gazebo)">
+      <!-- Keep Gazebo rendering tied to the same measured C10 calibration
+           used by the real usb_cam driver. -->
+      <xacro:property name="c10_calibration" value="${xacro.load_yaml('$(find wvcsc_c10_camera)/config/c10_intrinsics.yaml')}"/>
+      <xacro:property name="c10_width" value="${c10_calibration['image_width']}"/>
+      <xacro:property name="c10_height" value="${c10_calibration['image_height']}"/>
+      <xacro:property name="c10_fx" value="${c10_calibration['camera_matrix']['data'][0]}"/>
+      <xacro:property name="c10_fy" value="${c10_calibration['camera_matrix']['data'][4]}"/>
+      <xacro:property name="c10_cx" value="${c10_calibration['camera_matrix']['data'][2]}"/>
+      <xacro:property name="c10_cy" value="${c10_calibration['camera_matrix']['data'][5]}"/>
+      <xacro:property name="c10_k1" value="${c10_calibration['distortion_coefficients']['data'][0]}"/>
+      <xacro:property name="c10_k2" value="${c10_calibration['distortion_coefficients']['data'][1]}"/>
+      <xacro:property name="c10_p1" value="${c10_calibration['distortion_coefficients']['data'][2]}"/>
+      <xacro:property name="c10_p2" value="${c10_calibration['distortion_coefficients']['data'][3]}"/>
+      <xacro:property name="c10_k3" value="${c10_calibration['distortion_coefficients']['data'][4]}"/>
       <!-- Gazebo lumps fixed camera_link into link6, so attach its sensor to
            the retained parent link with the equivalent fixed transform. -->
@@ -138,12 +153,23 @@
           <pose>-0.055 0 0.05 0 -1.57079632679 0</pose>
           <camera name="c10_optical">
-            <horizontal_fov>1.8</horizontal_fov>
+            <horizontal_fov>${2.0 * atan(c10_width / (2.0 * c10_fx))}</horizontal_fov>
             <image>
-              <width>1280</width>
-              <height>720</height>
+              <width>${c10_width}</width>
+              <height>${c10_height}</height>
               <format>R8G8B8</format>
             </image>
             <clip><near>0.02</near><far>300</far></clip>
-            <noise><type>gaussian</type><mean>0.0</mean><stddev>0.007</stddev></noise>
+            <distortion>
+              <k1>${c10_k1}</k1><k2>${c10_k2}</k2><k3>${c10_k3}</k3>
+              <p1>${c10_p1}</p1><p2>${c10_p2}</p2>
+              <center>${c10_cx / c10_width} ${c10_cy / c10_height}</center>
+            </distortion>
+            <lens>
+              <intrinsics>
+                <fx>${c10_fx}</fx><fy>${c10_fy}</fy>
+                <cx>${c10_cx}</cx><cy>${c10_cy}</cy><s>0</s>
+              </intrinsics>
+            </lens>
+            <noise><type>gaussian</type><mean>0.0</mean><stddev>$(arg c10_noise_stddev)</stddev></noise>
           </camera>
           <plugin name="c10_camera_plugin" filename="libgazebo_ros_camera.so">
@@ -167,4 +193,11 @@
             <camera_name>color</camera_name>
             <frame_name>camera_color_optical_frame</frame_name>
+            <!-- gazebo_ros_camera publishes K with one focal length; retain
+                 measured fy in P while rendering uses the full fx/fy pair. -->
+            <focal_length>${c10_fx}</focal_length>
+            <cx>${c10_cx}</cx><cy>${c10_cy}</cy>
+            <P_fx>${c10_fx}</P_fx><P_fy>${c10_fy}</P_fy>
+            <P_cx>${c10_cx}</P_cx><P_cy>${c10_cy}</P_cy>
+            <border_crop>false</border_crop>
           </plugin>
         </sensor>
