Commit message: 2026 07.15

File: src/wvcsc_description/urdf/wvcsc_utb_alicia.urdf.xacro (robot description, xacro)
@@ -4,4 +4,9 @@
   <xacro:arg name="enable_ackermann" default="true"/>
   <xacro:arg name="enable_gazebo_ros2_control" default="false"/>
+  <xacro:arg name="enable_c10_camera" default="true"/>
+  <xacro:arg name="enable_c10_gazebo" default="false"/>
+  <!-- Temporary eye-in-hand extrinsics. Recalibrate after the real bracket is fixed. -->
+  <xacro:arg name="c10_mount_xyz" default="-0.055 0 -0.10"/>
+  <xacro:arg name="c10_mount_rpy" default="0 -1.57079632679 0"/>
   <xacro:arg name="gazebo_controllers_file" default="$(find wvcsc_description)/config/ros2_controllers.yaml"/>
   <xacro:arg name="ros2_control_plugin" default="mock_components/GenericSystem"/>
@@ -28,4 +33,102 @@
     <parent link="arm_mount_link"/><child link="alicia_base_link"/><origin xyz="0 0 0.06"/>
   </joint>
+  <!--
+    C10 eye-in-hand model. camera_link follows Gazebo's +X-forward camera
+    convention; camera_color_optical_frame follows REP-103 (+Z forward,
+    +X right, +Y down).  The optical axis and spray_nozzle_link +Z axis are
+    parallel, so IBVS only corrects image-plane X/Y and preserves spray range.
+  -->
+  <xacro:if value="$(arg enable_c10_camera)">
+    <link name="camera_link">
+      <visual>
+        <origin xyz="0 0 0" rpy="0 0 0"/>
+        <geometry>
+          <mesh filename="package://wvcsc_description/meshes/c10/camera.dae"/>
+        </geometry>
+      </visual>
+      <collision>
+        <origin xyz="0 0 0" rpy="0 0 0"/>
+        <geometry><box size="0.070 0.040 0.025"/></geometry>
+      </collision>
+      <inertial>
+        <mass value="0.130"/>
+        <inertia ixx="0.000020" ixy="0" ixz="0"
+                 iyy="0.000055" iyz="0" izz="0.000060"/>
+      </inertial>
+    </link>
+    <joint name="c10_mount_joint" type="fixed">
+      <parent link="tool0"/>
+      <child link="camera_link"/>
+      <origin xyz="$(arg c10_mount_xyz)" rpy="$(arg c10_mount_rpy)"/>
+    </joint>
+    <link name="camera_color_optical_frame"/>
+    <joint name="camera_color_optical_joint" type="fixed">
+      <parent link="camera_link"/>
+      <child link="camera_color_optical_frame"/>
+      <origin xyz="0 0 0" rpy="-1.57079632679 0 -1.57079632679"/>
+    </joint>
+    <link name="spray_nozzle_link">
+      <visual>
+        <origin xyz="0 0 0.025" rpy="0 0 0"/>
+        <geometry><cylinder radius="0.006" length="0.05"/></geometry>
+        <material name="nozzle_blue"><color rgba="0.05 0.15 0.8 1"/></material>
+      </visual>
+      <collision>
+        <origin xyz="0 0 0.025" rpy="0 0 0"/>
+        <geometry><cylinder radius="0.006" length="0.05"/></geometry>
+      </collision>
+      <inertial>
+        <mass value="0.03"/>
+        <inertia ixx="0.000006" ixy="0" ixz="0"
+                 iyy="0.000006" iyz="0" izz="0.000001"/>
+      </inertial>
+    </link>
+    <joint name="spray_nozzle_joint" type="fixed">
+      <parent link="tool0"/>
+      <child link="spray_nozzle_link"/>
+      <origin xyz="0 0 0.01" rpy="0 0 0"/>
+    </joint>
+    <xacro:if value="$(arg enable_c10_gazebo)">
+      <gazebo reference="camera_link">
+        <sensor name="c10_color" type="camera">
+          <always_on>true</always_on>
+          <update_rate>30.0</update_rate>
+          <visualize>true</visualize>
+          <camera name="c10_color">
+            <horizontal_fov>1.8</horizontal_fov>
+            <image>
+              <width>1280</width>
+              <height>720</height>
+              <format>R8G8B8</format>
+            </image>
+            <clip><near>0.02</near><far>300</far></clip>
+            <noise><type>gaussian</type><mean>0.0</mean><stddev>0.007</stddev></noise>
+          </camera>
+          <plugin name="c10_camera_plugin" filename="libgazebo_ros_camera.so">
+            <ros>
+              <namespace>/camera/camera</namespace>
+              <remapping>color/image_raw:=color/image_rect_raw</remapping>
+              <qos>
+                <topic name="color/image_rect_raw">
+                  <publisher>
+                    <reliability>best_effort</reliability>
+                    <history depth="1">keep_last</history>
+                  </publisher>
+                </topic>
+                <topic name="color/camera_info">
+                  <publisher>
+                    <reliability>best_effort</reliability>
+                    <history depth="1">keep_last</history>
+                  </publisher>
+                </topic>
+              </qos>
+            </ros>
+            <camera_name>color</camera_name>
+            <frame_name>camera_color_optical_frame</frame_name>
+          </plugin>
+        </sensor>
+      </gazebo>
+    </xacro:if>
+  </xacro:if>
   <xacro:if value="$(arg enable_arm_control)">
     <xacro:alicia_m_v1_1_follower_ros2_control

Commit message: 2026.07.16 1820

File: src/wvcsc_description/urdf/wvcsc_utb_alicia.urdf.xacro (robot description, xacro)
@@ -36,6 +36,5 @@
     C10 eye-in-hand model. camera_link follows Gazebo's +X-forward camera
     convention; camera_color_optical_frame follows REP-103 (+Z forward,
-    +X right, +Y down).  The optical axis and spray_nozzle_link +Z axis are
-    parallel, so IBVS only corrects image-plane X/Y and preserves spray range.
+    +X right, +Y down). tool0 is the temporary logical spray point.
   -->
   <xacro:if value="$(arg enable_c10_camera)">
@@ -67,25 +66,4 @@
       <child link="camera_color_optical_frame"/>
       <origin xyz="0 0 0" rpy="-1.57079632679 0 -1.57079632679"/>
-    </joint>
-    <link name="spray_nozzle_link">
-      <visual>
-        <origin xyz="0 0 0.025" rpy="0 0 0"/>
-        <geometry><cylinder radius="0.006" length="0.05"/></geometry>
-        <material name="nozzle_blue"><color rgba="0.05 0.15 0.8 1"/></material>
-      </visual>
-      <collision>
-        <origin xyz="0 0 0.025" rpy="0 0 0"/>
-        <geometry><cylinder radius="0.006" length="0.05"/></geometry>
-      </collision>
-      <inertial>
-        <mass value="0.03"/>
-        <inertia ixx="0.000006" ixy="0" ixz="0"
-                 iyy="0.000006" iyz="0" izz="0.000001"/>
-      </inertial>
-    </link>
-    <joint name="spray_nozzle_joint" type="fixed">
-      <parent link="tool0"/>
-      <child link="spray_nozzle_link"/>
-      <origin xyz="0 0 0.01" rpy="0 0 0"/>
     </joint>
     <xacro:if value="$(arg enable_c10_gazebo)">
@@ -145,5 +123,5 @@
   <gazebo reference="laser">
     <sensor name="laser" type="ray">
-      <always_on>true</always_on><update_rate>10</update_rate><visualize>true</visualize>
+      <always_on>true</always_on><update_rate>10</update_rate><visualize>false</visualize>
       <ray>
         <scan><horizontal><samples>720</samples><resolution>1</resolution><min_angle>-3.141592653589793</min_angle><max_angle>3.141592653589793</max_angle></horizontal></scan>

Commit message: 2026.07.21:02:29 完成喷嘴偏移补偿与Alicia-M自动手眼标定

File: src/wvcsc_description/urdf/wvcsc_utb_alicia.urdf.xacro (robot description, xacro)
@@ -9,4 +9,7 @@
   <xacro:arg name="c10_mount_xyz" default="-0.055 0 -0.10"/>
   <xacro:arg name="c10_mount_rpy" default="0 -1.57079632679 0"/>
+  <!-- Calibrated spray origin; local +Z is the liquid centreline. -->
+  <xacro:arg name="nozzle_mount_xyz" default="0 0 0"/>
+  <xacro:arg name="nozzle_mount_rpy" default="0 0 0"/>
   <xacro:arg name="gazebo_controllers_file" default="$(find wvcsc_description)/config/ros2_controllers.yaml"/>
   <xacro:arg name="ros2_control_plugin" default="mock_components/GenericSystem"/>
@@ -32,4 +35,10 @@
   <joint name="alicia_mount_joint" type="fixed">
     <parent link="arm_mount_link"/><child link="alicia_base_link"/><origin xyz="0 0 0.06"/>
+  </joint>
+  <link name="spray_nozzle_link"/>
+  <joint name="spray_nozzle_joint" type="fixed">
+    <parent link="tool0"/>
+    <child link="spray_nozzle_link"/>
+    <origin xyz="$(arg nozzle_mount_xyz)" rpy="$(arg nozzle_mount_rpy)"/>
   </joint>
   <!--

Commit message: 2026 07.21 23:09

File: src/wvcsc_description/urdf/wvcsc_utb_alicia.urdf.xacro (robot description, xacro)
@@ -6,4 +6,5 @@
   <xacro:arg name="enable_c10_camera" default="true"/>
   <xacro:arg name="enable_c10_gazebo" default="false"/>
+  <xacro:arg name="calibration_fix_base" default="false"/>
     <!-- 机械臂车顶安装参数 -->
   <!--
@@ -19,7 +20,7 @@
   <!--
     机械臂相对于车顶安装坐标系的位置：
-    沿 base_link 正 X 方向平移 0.10 m。
-  -->
-  <xacro:arg name="arm_mount_xyz" default="-0.20 0 0"/>
+    沿 base_link 负 X 方向平移 0.40 m。
+  -->
+  <xacro:arg name="arm_mount_xyz" default="-0.40 0 0"/>
   <!--
     绕 Z 轴旋转 180°，使机械臂底座 X 轴方向反转，
@@ -48,4 +49,12 @@
   <xacro:include filename="$(find alicia_m_descriptions)/urdf/Alicia_M_v1_1/Alicia_M_v1_1_follower.urdf"/>
   <xacro:include filename="$(find alicia_m_moveit_config)/config/alicia_m_v1_1_follower.ros2_control.xacro"/>
+  <xacro:if value="$(arg calibration_fix_base)">
+    <link name="world"/>
+    <joint name="world_to_base_footprint" type="fixed">
+      <parent link="world"/>
+      <child link="base_footprint"/>
+      <origin xyz="0 0 0" rpy="0 0 0"/>
+    </joint>
+  </xacro:if>
   <!--
     车顶安装坐标系。

Commit message: 2026 07.27 0200

File: src/wvcsc_description/urdf/wvcsc_utb_alicia.urdf.xacro (robot description, xacro)
@@ -89,5 +89,51 @@
       rpy="$(arg arm_mount_rpy)"/>
   </joint>
-  <link name="spray_nozzle_link"/>
+  <!-- 车顶广域喷洒柱：底面中心位于 base_link (0.10, 0, 0.675)。
+       该模型既是 Gazebo 中的广域喷洒出雾原点，也是 MoveIt 必须避开的
+       自碰撞实体；+Z 为柱体和环喷的轴线方向。 -->
+  <link name="wide_sprayer_link">
+    <visual>
+      <origin xyz="0 0 0.250" rpy="0 0 0"/>
+      <geometry><cylinder radius="0.030" length="0.500"/></geometry>
+      <material name="wide_sprayer_blue"><color rgba="0.08 0.24 0.34 1"/></material>
+    </visual>
+    <visual>
+      <origin xyz="0 0 0.500" rpy="0 0 0"/>
+      <geometry><cylinder radius="0.034" length="0.012"/></geometry>
+      <material name="wide_sprayer_cap"><color rgba="0.30 0.72 0.78 1"/></material>
+    </visual>
+    <collision>
+      <origin xyz="0 0 0.255" rpy="0 0 0"/>
+      <geometry><cylinder radius="0.035" length="0.510"/></geometry>
+    </collision>
+  </link>
+  <joint name="wide_sprayer_joint" type="fixed">
+    <parent link="base_link"/>
+    <child link="wide_sprayer_link"/>
+    <origin xyz="0.10 0 $(arg vehicle_roof_z)" rpy="0 0 0"/>
+  </joint>
+  <!-- tool0 即当前喷嘴安装基准；局部 +Z 为喷流中心轴。使用三级圆柱形成
+       紧凑的中空喷嘴外观，碰撞包络只略大于真实外观。 -->
+  <link name="spray_nozzle_link">
+    <visual>
+      <origin xyz="0 0 0.004" rpy="0 0 0"/>
+      <geometry><cylinder radius="0.011" length="0.008"/></geometry>
+      <material name="nozzle_mount"><color rgba="0.16 0.18 0.20 1"/></material>
+    </visual>
+    <visual>
+      <origin xyz="0 0 0.015" rpy="0 0 0"/>
+      <geometry><cylinder radius="0.009" length="0.014"/></geometry>
+      <material name="nozzle_brass"><color rgba="0.70 0.48 0.12 1"/></material>
+    </visual>
+    <visual>
+      <origin xyz="0 0 0.031" rpy="0 0 0"/>
+      <geometry><cylinder radius="0.005" length="0.010"/></geometry>
+      <material name="nozzle_exit"><color rgba="0.06 0.06 0.06 1"/></material>
+    </visual>
+    <collision>
+      <origin xyz="0 0 0.0175" rpy="0 0 0"/>
+      <geometry><cylinder radius="0.012" length="0.035"/></geometry>
+    </collision>
+  </link>
   <joint name="spray_nozzle_joint" type="fixed">
     <parent link="tool0"/>

Commit message: 2026 07.29 1533-小车导航参数调整

File: src/wvcsc_description/urdf/wvcsc_utb_alicia.urdf.xacro (robot description, xacro)
@@ -267,5 +267,5 @@
       <always_on>true</always_on><update_rate>10</update_rate><visualize>false</visualize>
       <ray>
-        <scan><horizontal><samples>720</samples><resolution>1</resolution><min_angle>-3.141592653589793</min_angle><max_angle>3.141592653589793</max_angle></horizontal></scan>
+        <scan><horizontal><samples>720</samples><resolution>1</resolution><min_angle>-1.047</min_angle><max_angle>1.047</max_angle></horizontal></scan>
         <range><min>0.15</min><max>20</max><resolution>0.02</resolution></range>
       </ray>

File: src/wvcsc_vehicle/wtb_car_driver/urdf/wtb_car.xacro (robot description, xacro)
@@ -10,6 +10,10 @@
   <xacro:property name="wheel_radius" value="0.20"/>
   <xacro:property name="wheel_length" value="0.12"/>
-  <xacro:property name="wheel_x" value="0.35"/>
-  <xacro:property name="wheel_y" value="0.43"/>
+  <!-- Measured vehicle geometry: front/rear axle distance is the wheelbase;
+       left/right wheel-center distance is the track width. -->
+  <xacro:property name="wheel_base" value="0.70"/>
+  <xacro:property name="track_width" value="0.86"/>
+  <xacro:property name="wheel_x" value="${wheel_base / 2.0}"/>
+  <xacro:property name="wheel_y" value="${track_width / 2.0}"/>
   <xacro:macro name="box_inertial" params="mass x y z">
     <inertial>
